File: EscaramujoExternalTL.sch (KiCad schematic (older format))
At the start: 24 parts, among them P1 CONN_01X03, U1 TL074

Commit message: Schematic and PCB design finished
Parts:
- removed R1, R2: 10k, Resistors_ThroughHole:Resistor_Horizontal_RM7mm, symbol R
- added R7, R8: 200, Resistors_ThroughHole:Resistor_Horizontal_RM7mm, symbol R
- R5, R6: value 10k -> 200
- renumbered R3 to R1, R4 to R2, R7 to R3, R8 to R4
Connections:
- net VEE: now also R5.1, R6.1, R7.1, R8.1; no longer RV1.1, RV2.1, RV3.1, RV4.1
- net at R1.2, U1.1: now also U1.2 (-)
- net at R3.2, U1.8: now also U1.9 (-); no longer R5.1
- net at R5.2: now also RV1.1; no longer U1.9 (-)
- net at U1.6 (-): now also R2.2, U1.7
- net at R6.2: now also RV2.1; no longer U1.13 (-)
- net at R4.2, U1.14: now also U1.13 (-); no longer R6.1
- new net: R7.2, RV3.1
- new net: R8.2, RV4.1
Changed lines of the file:
@@
 $EndComp
 $Comp
-L GND #PWR01
+L GND #PWR1
 U 1 1 57E2CC5B
 P 3500 2750
-F 0 "#PWR01" H 3500 2500 50  0001 C CNN
+F 0 "#PWR1" H 3500 2500 50  0001 C CNN
 F 1 "GND" H 3500 2600 50  0000 C CNN
 F 2 "" H 3500 2750 50  0000 C CNN
@@
 $EndComp
 $Comp
-L VCC #PWR02
+L VCC #PWR3
 U 1 1 57E2CC75
 P 4000 2850
-F 0 "#PWR02" H 4000 2700 50  0001 C CNN
+F 0 "#PWR3" H 4000 2700 50  0001 C CNN
 F 1 "VCC" H 4000 3000 50  0000 C CNN
 F 2 "" H 4000 2850 50  0000 C CNN
@@
 $EndComp
 $Comp
-L VEE #PWR03
+L VEE #PWR4
 U 1 1 57E2CC8F
 P 4000 3900
-F 0 "#PWR03" H 4000 3750 50  0001 C CNN
+F 0 "#PWR4" H 4000 3750 50  0001 C CNN
 F 1 "VEE" H 4000 4050 50  0000 C CNN
 F 2 "" H 4000 3900 50  0000 C CNN
@@
 	4000 2850 4000 3000
 $Comp
-L R R3
+L R R1
 U 1 1 57E2CE88
 P 4700 3300
-F 0 "R3" V 4780 3300 50  0000 C CNN
+F 0 "R1" V 4780 3300 50  0000 C CNN
 F 1 "200" V 4700 3300 50  0000 C CNN
 F 2 "Resistors_ThroughHole:Resistor_Horizontal_RM7mm" V 4630 3300 50  0001 C CNN
@@
 Wire Wire Line
 	4000 3600 4000 3900
-Wire Wire Line
-	3300 3450 3300 3850
-Wire Wire Line
-	3300 3850 4000 3850
 Connection ~ 4000 3850
-$Comp
-L R R1
-U 1 1 57E2D1C2
-P 3700 3650
-F 0 "R1" V 3780 3650 50  0000 C CNN
-F 1 "10k" V 3700 3650 50  0000 C CNN
-F 2 "Resistors_ThroughHole:Resistor_Horizontal_RM7mm" V 3630 3650 50  0001 C CNN
-F 3 "" H 3700 3650 50  0000 C CNN
-	1    3700 3650
-	0    1    1    0
-$EndComp
 Wire Wire Line
 	3800 3400 3500 3400
@@
 	3500 3400 3500 3650
 Wire Wire Line
-	3500 3650 3550 3650
-Wire Wire Line
-	3850 3650 4450 3650
+	3500 3650 4450 3650
 Wire Wire Line
 	4450 3650 4450 3300
@@
 $EndComp
 $Comp
-L GND #PWR04
+L GND #PWR7
 U 1 1 57E2D51D
 P 6100 2700
-F 0 "#PWR04" H 6100 2450 50  0001 C CNN
+F 0 "#PWR7" H 6100 2450 50  0001 C CNN
 F 1 "GND" H 6100 2550 50  0000 C CNN
 F 2 "" H 6100 2700 50  0000 C CNN
@@
 $EndComp
 $Comp
-L VCC #PWR05
+L VCC #PWR9
 U 1 1 57E2D523
 P 6600 2800
-F 0 "#PWR05" H 6600 2650 50  0001 C CNN
+F 0 "#PWR9" H 6600 2650 50  0001 C CNN
 F 1 "VCC" H 6600 2950 50  0000 C CNN
 F 2 "" H 6600 2800 50  0000 C CNN
@@
 $EndComp
 $Comp
-L VEE #PWR06
+L VEE #PWR10
 U 1 1 57E2D529
 P 6600 3850
-F 0 "#PWR06" H 6600 3700 50  0001 C CNN
+F 0 "#PWR10" H 6600 3700 50  0001 C CNN
 F 1 "VEE" H 6600 4000 50  0000 C CNN
 F 2 "" H 6600 3850 50  0000 C CNN
@@
 	6600 2800 6600 2950
 $Comp
-L R R7
+L R R3
 U 1 1 57E2D530
 P 7300 3250
-F 0 "R7" V 7380 3250 50  0000 C CNN
+F 0 "R3" V 7380 3250 50  0000 C CNN
 F 1 "200" V 7300 3250 50  0000 C CNN
 F 2 "Resistors_ThroughHole:Resistor_Horizontal_RM7mm" V 7230 3250 50  0001 C CNN
@@
 Wire Wire Line
 	6600 3550 6600 3850
-Wire Wire Line
-	5900 3400 5900 3800
-Wire Wire Line
-	5900 3800 6600 3800
 Connection ~ 6600 3800
-$Comp
-L R R5
-U 1 1 57E2D54A
-P 6300 3600
-F 0 "R5" V 6380 3600 50  0000 C CNN
-F 1 "10k" V 6300 3600 50  0000 C CNN
-F 2 "Resistors_ThroughHole:Resistor_Horizontal_RM7mm" V 6230 3600 50  0001 C CNN
-F 3 "" H 6300 3600 50  0000 C CNN
-	1    6300 3600
-	0    1    1    0
-$EndComp
 Wire Wire Line
 	6400 3350 6100 3350
@@
 	6100 3350 6100 3600
 Wire Wire Line
-	6100 3600 6150 3600
-Wire Wire Line
-	6450 3600 7050 3600
+	6100 3600 7050 3600
 Wire Wire Line
 	7050 3600 7050 3250
@@
 $EndComp
 $Comp
-L GND #PWR07
+L GND #PWR2
 U 1 1 57E2DA18
 P 3500 4400
-F 0 "#PWR07" H 3500 4150 50  0001 C CNN
+F 0 "#PWR2" H 3500 4150 50  0001 C CNN
 F 1 "GND" H 3500 4250 50  0000 C CNN
 F 2 "" H 3500 4400 50  0000 C CNN
@@
 $EndComp
 $Comp
-L VCC #PWR08
+L VCC #PWR5
 U 1 1 57E2DA1E
 P 4000 4500
-F 0 "#PWR08" H 4000 4350 50  0001 C CNN
+F 0 "#PWR5" H 4000 4350 50  0001 C CNN
 F 1 "VCC" H 4000 4650 50  0000 C CNN
 F 2 "" H 4000 4500 50  0000 C CNN
@@
 $EndComp
 $Comp
-L VEE #PWR09
+L VEE #PWR6
 U 1 1 57E2DA24
 P 4000 5550
-F 0 "#PWR09" H 4000 5400 50  0001 C CNN
+F 0 "#PWR6" H 4000 5400 50  0001 C CNN
 F 1 "VEE" H 4000 5700 50  0000 C CNN
 F 2 "" H 4000 5550 50  0000 C CNN
@@
 	4000 4500 4000 4650
 $Comp
-L R R4
+L R R2
 U 1 1 57E2DA2B
 P 4700 4950
-F 0 "R4" V 4780 4950 50  0000 C CNN
+F 0 "R2" V 4780 4950 50  0000 C CNN
 F 1 "200" V 4700 4950 50  0000 C CNN
 F 2 "Resistors_ThroughHole:Resistor_Horizontal_RM7mm" V 4630 4950 50  0001 C CNN
@@
 Wire Wire Line
 	4000 5250 4000 5550
-Wire Wire Line
-	3300 5100 3300 5500
-Wire Wire Line
-	3300 5500 4000 5500
 Connection ~ 4000 5500
-$Comp
-L R R2
-U 1 1 57E2DA45
-P 3700 5300
-F 0 "R2" V 3780 5300 50  0000 C CNN
-F 1 "10k" V 3700 5300 50  0000 C CNN
-F 2 "Resistors_ThroughHole:Resistor_Horizontal_RM7mm" V 3630 5300 50  0001 C CNN
-F 3 "" H 3700 5300 50  0000 C CNN
-	1    3700 5300
-	0    1    1    0
-$EndComp
 Wire Wire Line
 	3800 5050 3500 5050
@@
 	3500 5050 3500 5300
 Wire Wire Line
-	3500 5300 3550 5300
-Wire Wire Line
-	3850 5300 4450 5300
+	3500 5300 4450 5300
 Wire Wire Line
 	4450 5300 4450 4950
@@
 $EndComp
 $Comp
-L GND #PWR010
+L GND #PWR8
 U 1 1 57E2DA63
 P 6100 4350
-F 0 "#PWR010" H 6100 4100 50  0001 C CNN
+F 0 "#PWR8" H 6100 4100 50  0001 C CNN
 F 1 "GND" H 6100 4200 50  0000 C CNN
 F 2 "" H 6100 4350 50  0000 C CNN
@@
 $EndComp
 $Comp
-L VCC #PWR011
+L VCC #PWR11
 U 1 1 57E2DA69
 P 6600 4450
-F 0 "#PWR011" H 6600 4300 50  0001 C CNN
+F 0 "#PWR11" H 6600 4300 50  0001 C CNN
 F 1 "VCC" H 6600 4600 50  0000 C CNN
 F 2 "" H 6600 4450 50  0000 C CNN
@@
 $EndComp
 $Comp
-L VEE #PWR012
+L VEE #PWR12
 U 1 1 57E2DA6F
 P 6600 5500
-F 0 "#PWR012" H 6600 5350 50  0001 C CNN
+F 0 "#PWR12" H 6600 5350 50  0001 C CNN
 F 1 "VEE" H 6600 5650 50  0000 C CNN
 F 2 "" H 6600 5500 50  0000 C CNN
@@
 	6600 4450 6600 4600
 $Comp
-L R R8
+L R R4
 U 1 1 57E2DA76
 P 7300 4900
-F 0 "R8" V 7380 4900 50  0000 C CNN
+F 0 "R4" V 7380 4900 50  0000 C CNN
 F 1 "200" V 7300 4900 50  0000 C CNN
 F 2 "Resistors_ThroughHole:Resistor_Horizontal_RM7mm" V 7230 4900 50  0001 C CNN
@@
 Wire Wire Line
 	6600 5200 6600 5500
-Wire Wire Line
-	5900 5050 5900 5450
-Wire Wire Line
-	5900 5450 6600 5450
 Connection ~ 6600 5450
-$Comp
-L R R6
-U 1 1 57E2DA90
-P 6300 5250
-F 0 "R6" V 6380 5250 50  0000 C CNN
-F 1 "10k" V 6300 5250 50  0000 C CNN
-F 2 "Resistors_ThroughHole:Resistor_Horizontal_RM7mm" V 6230 5250 50  0001 C CNN
-F 3 "" H 6300 5250 50  0000 C CNN
-	1    6300 5250
-	0    1    1    0
-$EndComp
 Wire Wire Line
 	6400 5000 6100 5000
@@
 	6100 5000 6100 5250
 Wire Wire Line
-	6100 5250 6150 5250
-Wire Wire Line
-	6450 5250 7050 5250
+	6100 5250 7050 5250
 Wire Wire Line
 	7050 5250 7050 4900
 Connection ~ 7050 4900
 $Comp
-L VCC #PWR013
+L VCC #PWR16
 U 1 1 57E2E6AC
 P 8500 3850
-F 0 "#PWR013" H 8500 3700 50  0001 C CNN
+F 0 "#PWR16" H 8500 3700 50  0001 C CNN
 F 1 "VCC" H 8500 4000 50  0000 C CNN
 F 2 "" H 8500 3850 50  0000 C CNN
@@
 $EndComp
 $Comp
-L VEE #PWR014
+L VEE #PWR18
 U 1 1 57E2E6FF
 P 8900 3850
-F 0 "#PWR014" H 8900 3700 50  0001 C CNN
+F 0 "#PWR18" H 8900 3700 50  0001 C CNN
 F 1 "VEE" H 8900 4000 50  0000 C CNN
 F 2 "" H 8900 3850 50  0000 C CNN
@@
 $EndComp
 $Comp
-L GND #PWR015
+L GND #PWR17
 U 1 1 57E2E752
 P 8700 3850
-F 0 "#PWR015" H 8700 3600 50  0001 C CNN
+F 0 "#PWR17" H 8700 3600 50  0001 C CNN
 F 1 "GND" H 8700 3700 50  0000 C CNN
 F 2 "" H 8700 3850 50  0000 C CNN
@@
 	7950 4300 7950 4150
 $Comp
-L GND #PWR016
+L GND #PWR14
 U 1 1 57E31284
 P 7800 4350
-F 0 "#PWR016" H 7800 4100 50  0001 C CNN
+F 0 "#PWR14" H 7800 4100 50  0001 C CNN
 F 1 "GND" H 7800 4200 50  0000 C CNN
 F 2 "" H 7800 4350 50  0000 C CNN
@@
 Connection ~ 7800 4300
 $Comp
-L VCC #PWR017
+L VCC #PWR13
 U 1 1 57E313C8
 P 7650 3750
-F 0 "#PWR017" H 7650 3600 50  0001 C CNN
+F 0 "#PWR13" H 7650 3600 50  0001 C CNN
 F 1 "VCC" H 7650 3900 50  0000 C CNN
 F 2 "" H 7650 3750 50  0000 C CNN
@@
 $EndComp
 $Comp
-L VEE #PWR018
+L VEE #PWR15
 U 1 1 57E31424
 P 7950 3750
-F 0 "#PWR018" H 7950 3600 50  0001 C CNN
+F 0 "#PWR15" H 7950 3600 50  0001 C CNN
 F 1 "VEE" H 7950 3900 50  0000 C CNN
 F 2 "" H 7950 3750 50  0000 C CNN
@@
 Wire Wire Line
 	7950 3750 7950 3850
+$Comp
+L R R5
+U 1 1 57E3291E
+P 3550 3850
+F 0 "R5" V 3630 3850 50  0000 C CNN
+F 1 "200" V 3550 3850 50  0000 C CNN
+F 2 "Resistors_ThroughHole:Resistor_Horizontal_RM7mm" V 3480 3850 50  0001 C CNN
+F 3 "" H 3550 3850 50  0000 C CNN
+	1    3550 3850
+	0    1    1    0
+$EndComp
+$Comp
+L R R7
+U 1 1 57E329A4
+P 6200 3800
+F 0 "R7" V 6280 3800 50  0000 C CNN
+F 1 "200" V 6200 3800 50  0000 C CNN
+F 2 "Resistors_ThroughHole:Resistor_Horizontal_RM7mm" V 6130 3800 50  0001 C CNN
+F 3 "" H 6200 3800 50  0000 C CNN
+	1    6200 3800
+	0    1    1    0
+$EndComp
+$Comp
+L R R8
+U 1 1 57E32A51
+P 6200 5450
+F 0 "R8" V 6280 5450 50  0000 C CNN
+F 1 "200" V 6200 5450 50  0000 C CNN
+F 2 "Resistors_ThroughHole:Resistor_Horizontal_RM7mm" V 6130 5450 50  0001 C CNN
+F 3 "" H 6200 5450 50  0000 C CNN
+	1    6200 5450
+	0    1    1    0
+$EndComp
+$Comp
+L R R6
+U 1 1 57E32C0D
+P 3600 5500
+F 0 "R6" V 3680 5500 50  0000 C CNN
+F 1 "200" V 3600 5500 50  0000 C CNN
+F 2 "Resistors_ThroughHole:Resistor_Horizontal_RM7mm" V 3530 5500 50  0001 C CNN
+F 3 "" H 3600 5500 50  0000 C CNN
+	1    3600 5500
+	0    1    1    0
+$EndComp
+Wire Wire Line
+	3750 5500 4000 5500
+Wire Wire Line
+	3450 5500 3300 5500
+Wire Wire Line
+	3300 5500 3300 5100
+Wire Wire Line
+	6050 5450 5900 5450
+Wire Wire Line
+	5900 5450 5900 5050
+Wire Wire Line
+	6350 5450 6600 5450
+Wire Wire Line
+	6350 3800 6600 3800
+Wire Wire Line
+	6050 3800 5900 3800
+Wire Wire Line
+	5900 3800 5900 3400
+Wire Wire Line
+	3700 3850 4000 3850
+Wire Wire Line
+	3400 3850 3300 3850
+Wire Wire Line
+	3300 3850 3300 3450
 $EndSCHEMATC
